File: Main_PCB/init/_saved_init.sch (KiCad schematic (older format))
At the start: 16 parts, among them J1 Conn_01x06_Male, J2 Conn_01x02_Male, J3 Conn_01x02_Female, J4 Conn_01x02_Female, J5 Conn_01x04_Female, U1 L293D

Commit message: modif du routage
Parts:
- D3: footprint Diode_THT:D_5KPW_P12.70mm_Horizontal -> Diode_THT:D_DO-41_SOD81_P10.16mm_Horizontal
Changed lines of the file:
@@
 F 0 "D3" H 2500 3650 50  0000 C CNN
 F 1 "1N4007" H 2500 3750 50  0000 C CNN
-F 2 "Diode_THT:D_5KPW_P12.70mm_Horizontal" H 2500 3900 50  0001 C CNN
+F 2 "Diode_THT:D_DO-41_SOD81_P10.16mm_Horizontal" H 2500 3900 50  0001 C CNN
 F 3 "~" H 2500 3900 50  0001 C CNN
 	1    2500 3900
