File: Main_PCB/init/init.kicad_pcb (KiCad board)
At the start: 2 copper layers, 70 x 50 mm, 15 parts, among them J1 Conn_01x06_Male, J2 Conn_01x02_Male, J3 Conn_01x02_Female, J4 Conn_01x02_Female, J5 Conn_01x04_Female, U1 L293D

Commit message: modif du routage
Parts:
- added D3: 1N4007, Diode_THT:D_DO-41_SOD81_P10.16mm_Horizontal, F.Cu at (77.5, 103.5)
- moved J2 2.34 mm to (80.0, 108.0)
Connections:
- J2 pad 1: +BATT -> Net-(D3-Pad2)
- U1 pad 8: +5V -> +BATT
Routing:
- net +BATT: track 10.6 -> 21.3 mm, vias 0 -> 2
- net Net-(D3-Pad2): track 0.00 -> 10.3 mm
- net +5V: track 171.9 -> 163.2 mm
- net GND: track 247.7 -> 247.0 mm
